File: Adafruit ST7565.sch (EAGLE design)
At the start: 19 parts, among them IC1 4050D, IC2 L4931D-GNDPIN7, Q3 2N7002, Q4 2N7002, SW1 ROTARTY_ENCODER, U1 SD_CARD_SOCKET

Commit message: Rev B
Parts:
- removed BLUE: Blue, SparkFun-Passives:JUMPER-PAD-2-NC_BY_TRACE
- removed GREEN: Green, SparkFun-Passives:JUMPER-PAD-2-NC_BY_TRACE
- removed RED: Red, SparkFun-Passives:JUMPER-PAD-2-NC_BY_TRACE
- removed U$1: 1X11_2MM, elb:1X11_2MM
- added B: Blue, SparkFun-Passives:JUMPER-PAD-2-NC_BY_TRACE
- added G: Green, SparkFun-Passives:JUMPER-PAD-2-NC_BY_TRACE
- added JP3: 1X11_2MM, elb:1X11_2MM
- added Q1, Q2: 2N7002, SparkFun-DiscreteSemi:MOSFET-NCHANNELBSS123LT1G
- added R: Red, SparkFun-Passives:JUMPER-PAD-2-NC_BY_TRACE
- added R3, R4: 4.7k, SparkFun-Passives:RESISTOR1206
- C1: value 1 uF -> 0.1uF
- C3: value 0.1uF -> 1 uF
- IC1: value 4050D -> L4931D; device 40xx:4050D -> v-reg-3:L4931D-GNDPIN7
- IC2: value L4931D-GNDPIN7 -> 4050D; device v-reg-3:L4931D-GNDPIN7 -> 40xx:4050D
- renumbered C4 to C2
Connections:
- removed net N$6: GREEN.2, U$1.P$10
- removed net N$7: BLUE.2, U$1.P$11
- new net D17: JP1.8, Q4.G, R4.2
- new net D25: JP1.5, Q3.G, R3.2
- new net N$3: B.2, JP3.P$11
- new net N$4: G.2, JP3.P$10, Q3.D
- net +3.3V: now also C3.1, IC1.VOUT, IC2P.VDD, JP3.P$2, JP3.P$6, JP3.P$9; no longer C1.1, IC1P.VDD, IC2.VOUT, U$1.P$2, U$1.P$6, U$1.P$9
- net +5V: now also C1.1, IC1.VIN, SG1.+; no longer C3.1, IC2.VIN, SG1.-
- net D23: now also Q1.G; no longer Q3.G
- net D27: now also IC2B.I; no longer IC1B.I
- net D29: now also IC2A.I; no longer IC1A.I
- net D33: now also Q2.G; no longer Q4.G
- net D51: now also IC2C.I; no longer IC1C.I
- net D52: now also IC2E.I; no longer IC1E.I
- net D53: now also IC2D.I; no longer IC1D.I
- net GND: now also IC1.GND, IC2F.I, IC2P.VSS, JP2.2, JP3.P$7, Q1.S, Q2.S, R3.1, R4.1; no longer IC1F.I, IC1P.VSS, IC2.GND, U$1.P$7
- net LCD_A0: now also IC2B.O, JP3.P$3; no longer IC1B.O, U$1.P$3
- net LCD_CS: now also IC2A.O, JP3.P$1; no longer IC1A.O, U$1.P$1
- net MOSI: now also IC2C.O, JP3.P$5; no longer IC1C.O, U$1.P$5
- net N$1: now also Q1.D, SG1.-; no longer Q3.D, SG1.+
- net N$2: now also B.1, G.1, Q2.D, R.1; no longer BLUE.1, GREEN.1, Q4.D, RED.1
- net N$5: now also JP3.P$8, Q4.D, R.2; no longer RED.2, U$1.P$8
- net SCLK: now also IC2E.O, JP3.P$4; no longer IC1E.O, U$1.P$4
- net SD_CS: now also IC2D.O; no longer IC1D.O
Other:
- moved on the sheet: C1, C3, Q3, Q4, R2, SG1, U1
